Commit message: 解决scara抖动，以及小车适配问题

File: urdf/scara_robot.urdf (robot description, URDF)
Before this commit: robot scara_robot, 9 links, 8 joints
Joints:
- joint gripper_joint: limit lower=-0.15 upper=0.0 effort=100 velocity=100 -> lower=-0.15 upper=0.15 effort=100 velocity=100

Commit message: last update

File: urdf/scara_robot.urdf (robot description, URDF)
Before this commit: robot scara_robot, 9 links, 8 joints
Links:
- link finger1: geometry collision box size=0.02 0.002 0.02; visual box size=0.02 0.002 0.02
- link finger2: geometry collision box size=0.002 0.02 0.02; visual box size=0.002 0.02 0.02
- link finger3: geometry collision box size=0.02 0.002 0.02; visual box size=0.02 0.002 0.02
- link finger4: geometry collision box size=0.002 0.02 0.02; visual box size=0.002 0.02 0.02
Joints:
- joint finger1_joint: limit lower=-0.02 upper=0.0 effort=100 velocity=100 -> lower=-0.025 upper=0.0 effort=100 velocity=100
- joint finger2_joint: limit lower=0.0 upper=0.02 effort=100 velocity=100 -> lower=0.0 upper=0.025 effort=100 velocity=100
- joint finger3_joint: limit lower=0.0 upper=0.02 effort=100 velocity=100 -> lower=0.0 upper=0.025 effort=100 velocity=100
- joint finger4_joint: limit lower=-0.02 upper=0.0 effort=100 velocity=100 -> lower=-0.025 upper=0.0 effort=100 velocity=100
